File: serial-io.sch (KiCad schematic (older format))
At the start: 13 parts

Commit message: Crowbar updates and ERC fixes
This updates the Crowbar bus connectors and the layout of the
schematic to match the finalized pinouts. It also corrects an
error in the original schematic where the buses were not
properly routing due to lack of labels.

Finally, this change includes fixes for the ERC and adds the CPU
and RTC crystals to the system.
Parts:
- gave numbers to parts that had none: 13
Other:
- note added: "Note: ZDI debug header is in the backplane\nsheet!"
- note removed: "Note: JTAG debug header is in the backplane\nsheet!"
Changed lines of the file:
@@
 EESchema Schematic File Version 4
+LIBS:Zippy-cache
 EELAYER 29 0
 EELAYER END
@@
 $EndDescr
 Wire Wire Line
-	8050 3200 7650 3200
-Wire Wire Line
-	8050 3300 7650 3300
-Wire Wire Line
-	8050 3400 7650 3400
-Wire Wire Line
-	8050 3500 7650 3500
-NoConn ~ 8050 3900
-$Comp
-L eZ80:EZ80L92AZ050SG U?
+	8150 1500 7750 1500
+Wire Wire Line
+	8150 1600 7750 1600
+Wire Wire Line
+	8150 1700 7750 1700
+Wire Wire Line
+	8150 1800 7750 1800
+NoConn ~ 8150 2200
+$Comp
+L eZ80:EZ80L92AZ050SG U1
 U 2 1 5DA1F770
-P 8750 3600
-F 0 "U?" H 9280 3696 50  0000 L CNN
-F 1 "EZ80L92AZ050SG" H 9280 3605 50  0000 L CNN
-F 2 "QFP50P1600X1600X160-100N" H 8750 3600 50  0001 L BNN
-F 3 "" H 8750 3600 50  0001 L BNN
-F 4 "None" H 8750 3600 50  0001 L BNN "Field4"
-F 5 "EZ80L92AZ050SG" H 8750 3600 50  0001 L BNN "Field5"
-F 6 "LQFP-100 Zilog" H 8750 3600 50  0001 L BNN "Field6"
-F 7 "EZ80L92 Series 50 MHz IC WEBSERVER SMT eZ80 Microcontroller - LQFP-100" H 8750 3600 50  0001 L BNN "Field7"
-F 8 "Zilog" H 8750 3600 50  0001 L BNN "Field8"
-	2    8750 3600
-	1    0    0    -1
-$EndComp
-NoConn ~ 8050 3800
-NoConn ~ 8050 3700
-NoConn ~ 8050 3600
-Text Label 7650 3200 0    50   ~ 0
+P 8850 1900
+F 0 "U1" H 9380 1996 50  0000 L CNN
+F 1 "EZ80L92AZ050SG" H 9380 1905 50  0000 L CNN
+F 2 "QFP50P1600X1600X160-100N" H 8850 1900 50  0001 L BNN
+F 3 "" H 8850 1900 50  0001 L BNN
+F 4 "None" H 8850 1900 50  0001 L BNN "Field4"
+F 5 "EZ80L92AZ050SG" H 8850 1900 50  0001 L BNN "Field5"
+F 6 "LQFP-100 Zilog" H 8850 1900 50  0001 L BNN "Field6"
+F 7 "EZ80L92 Series 50 MHz IC WEBSERVER SMT eZ80 Microcontroller - LQFP-100" H 8850 1900 50  0001 L BNN "Field7"
+F 8 "Zilog" H 8850 1900 50  0001 L BNN "Field8"
+	2    8850 1900
+	1    0    0    -1
+$EndComp
+NoConn ~ 8150 2100
+NoConn ~ 8150 2000
+NoConn ~ 8150 1900
+Text Label 7750 1500 0    50   ~ 0
 CPU_TXD
-Text Label 7650 3300 0    50   ~ 0
+Text Label 7750 1600 0    50   ~ 0
 CPU_RXD
-Text Label 7650 3400 0    50   ~ 0
+Text Label 7750 1700 0    50   ~ 0
 CPU_RTS
-Text Label 7650 3500 0    50   ~ 0
+Text Label 7750 1800 0    50   ~ 0
 CPU_CTS
 Wire Wire Line
@@
 	4150 4200 4250 4200
 $Comp
-L power:GND #PWR?
+L power:GND #PWR0143
 U 1 1 5DA2C8E6
 P 4050 4250
-F 0 "#PWR?" H 4050 4000 50  0001 C CNN
+F 0 "#PWR0143" H 4050 4000 50  0001 C CNN
 F 1 "GND" H 4055 4077 50  0000 C CNN
 F 2 "" H 4050 4250 50  0001 C CNN
@@
 	4050 4200 4050 4250
 $Comp
-L power:GND #PWR?
+L power:GND #PWR0144
 U 1 1 5DA2D9A9
 P 5350 3050
-F 0 "#PWR?" H 5350 2800 50  0001 C CNN
+F 0 "#PWR0144" H 5350 2800 50  0001 C CNN
 F 1 "GND" H 5355 2877 50  0000 C CNN
 F 2 "" H 5350 3050 50  0001 C CNN
@@
 $EndComp
 $Comp
-L Device:C_Small C?
+L Device:C_Small C28
 U 1 1 5DA2E0A3
 P 5350 2950
-F 0 "C?" H 5442 2996 50  0000 L CNN
+F 0 "C28" H 5442 2996 50  0000 L CNN
 F 1 "100nF" H 5442 2905 50  0000 L CNN
 F 2 "" H 5350 2950 50  0001 C CNN
@@
 NoConn ~ 4450 2800
 $Comp
-L Connector:USB_B_Micro J?
+L Connector:USB_B_Micro J4
 U 1 1 5DA310C5
 P 1850 2500
-F 0 "J?" H 1907 2967 50  0000 C CNN
+F 0 "J4" H 1907 2967 50  0000 C CNN
 F 1 "USB_B_Micro" H 1907 2876 50  0000 C CNN
 F 2 "" H 2000 2450 50  0001 C CNN
@@
 $EndComp
 NoConn ~ 1750 2900
-Wire Wire Line
-	1850 2900 1850 2950
-Wire Wire Line
-	1850 2950 2150 2950
-$Comp
-L power:GND #PWR?
+$Comp
+L power:GND #PWR0145
 U 1 1 5DA343C0
 P 1850 3100
-F 0 "#PWR?" H 1850 2850 50  0001 C CNN
+F 0 "#PWR0145" H 1850 2850 50  0001 C CNN
 F 1 "GND" H 1855 2927 50  0000 C CNN
 F 2 "" H 1850 3100 50  0001 C CNN
@@
 Wire Wire Line
 	2150 2600 3350 2600
-Wire Wire Line
-	2150 2700 2150 2950
-$Comp
-L Device:R_Small_US R?
+$Comp
+L Device:R_Small_US R8
 U 1 1 5DA426C5
 P 2400 2100
-F 0 "R?" H 2468 2146 50  0000 L CNN
+F 0 "R8" H 2468 2146 50  0000 L CNN
 F 1 "4.7K" H 2468 2055 50  0000 L CNN
 F 2 "" H 2400 2100 50  0001 C CNN
@@
 $EndComp
 $Comp
-L Device:R_Small_US R?
+L Device:R_Small_US R7
 U 1 1 5DA451B2
 P 2400 1700
-F 0 "R?" H 2468 1746 50  0000 L CNN
+F 0 "R7" H 2468 1746 50  0000 L CNN
 F 1 "10K" H 2468 1655 50  0000 L CNN
 F 2 "" H 2400 1700 50  0001 C CNN
@@
 $EndComp
 $Comp
-L power:GND #PWR?
+L power:GND #PWR0146
 U 1 1 5DA45E16
 P 2400 1550
-F 0 "#PWR?" H 2400 1300 50  0001 C CNN
+F 0 "#PWR0146" H 2400 1300 50  0001 C CNN
 F 1 "GND" H 2405 1377 50  0000 C CNN
 F 2 "" H 2400 1550 50  0001 C CNN
@@
 SER_RES
 Wire Wire Line
-	1850 3100 1850 2950
-Connection ~ 1850 2950
-Wire Wire Line
 	4450 2700 5350 2700
 Wire Wire Line
@@
 SER_D-
 $Comp
-L power:+5V #PWR?
+L power:+5V #PWR0147
 U 1 1 5DA522B9
 P 3850 1900
-F 0 "#PWR?" H 3850 1750 50  0001 C CNN
+F 0 "#PWR0147" H 3850 1750 50  0001 C CNN
 F 1 "+5V" H 3865 2073 50  0000 C CNN
 F 2 "" H 3850 1900 50  0001 C CNN
@@
 $EndComp
 $Comp
-L Device:C_Small C?
+L Device:C_Small C25
 U 1 1 5DB6E529
 P 3650 4750
-F 0 "C?" H 3742 4796 50  0000 L CNN
+F 0 "C25" H 3742 4796 50  0000 L CNN
 F 1 "100nF" H 3742 4705 50  0000 L CNN
 F 2 "" H 3650 4750 50  0001 C CNN
@@
 $EndComp
 $Comp
-L Device:C_Small C?
+L Device:C_Small C26
 U 1 1 5DB7033D
 P 4100 4750
-F 0 "C?" H 4192 4796 50  0000 L CNN
+F 0 "C26" H 4192 4796 50  0000 L CNN
 F 1 "100nF" H 4192 4705 50  0000 L CNN
 F 2 "" H 4100 4750 50  0001 C CNN
@@
 $EndComp
 $Comp
-L Device:CP1_Small C?
+L Device:CP1_Small C27
 U 1 1 5DB7146D
 P 4550 4750
-F 0 "C?" H 4641 4796 50  0000 L CNN
+F 0 "C27" H 4641 4796 50  0000 L CNN
 F 1 "4.7uF" H 4641 4705 50  0000 L CNN
 F 2 "" H 4550 4750 50  0001 C CNN
@@
 	4100 4850 3650 4850
 $Comp
-L power:GND #PWR?
+L power:GND #PWR0148
 U 1 1 5DB72CE9
 P 3350 4850
-F 0 "#PWR?" H 3350 4600 50  0001 C CNN
+F 0 "#PWR0148" H 3350 4600 50  0001 C CNN
 F 1 "GND" H 3355 4677 50  0000 C CNN
 F 2 "" H 3350 4850 50  0001 C CNN
@@
 $EndComp
 $Comp
-L power:+5V #PWR?
+L power:+5V #PWR0149
 U 1 1 5DB7341B
 P 3350 4650
-F 0 "#PWR?" H 3350 4500 50  0001 C CNN
+F 0 "#PWR0149" H 3350 4500 50  0001 C CNN
 F 1 "+5V" H 3365 4823 50  0000 C CNN
 F 2 "" H 3350 4650 50  0001 C CNN
@@
 ~TXLED
 $Comp
-L Device:LED D?
+L Device:LED D1
 U 1 1 5DB7CACD
 P 2250 6350
-F 0 "D?" H 2243 6095 50  0000 C CNN
+F 0 "D1" H 2243 6095 50  0000 C CNN
 F 1 "RED" H 2243 6186 50  0000 C CNN
 F 2 "" H 2250 6350 50  0001 C CNN
@@
 $EndComp
 $Comp
-L Device:LED D?
+L Device:LED D2
 U 1 1 5DB7DCC6
 P 2250 6750
-F 0 "D?" H 2243 6495 50  0000 C CNN
+F 0 "D2" H 2243 6495 50  0000 C CNN
 F 1 "GREEN" H 2243 6586 50  0000 C CNN
 F 2 "" H 2250 6750 50  0001 C CNN
@@
 ~RXLED
 $Comp
-L Device:R_Small_US R?
+L Device:R_Small_US R6
 U 1 1 5DB81B16
 P 1800 6750
-F 0 "R?" V 1595 6750 50  0000 C CNN
+F 0 "R6" V 1595 6750 50  0000 C CNN
 F 1 "270" V 1686 6750 50  0000 C CNN
 F 2 "" H 1800 6750 50  0001 C CNN
@@
 $EndComp
 $Comp
-L Device:R_Small_US R?
+L Device:R_Small_US R5
 U 1 1 5DB823EE
 P 1800 6350
-F 0 "R?" V 1595 6350 50  0000 C CNN
+F 0 "R5" V 1595 6350 50  0000 C CNN
 F 1 "270" V 1686 6350 50  0000 C CNN
 F 2 "" H 1800 6350 50  0001 C CNN
@@
 Connection ~ 1550 6350
 $Comp
-L power:+5V #PWR?
+L power:+5V #PWR0150
 U 1 1 5DB86C1D
 P 1550 6150
-F 0 "#PWR?" H 1550 6000 50  0001 C CNN
+F 0 "#PWR0150" H 1550 6000 50  0001 C CNN
 F 1 "+5V" H 1565 6323 50  0000 C CNN
 F 2 "" H 1550 6150 50  0001 C CNN
@@
 NoConn ~ 3350 3200
 $Comp
-L dk_Interface-Controllers:FT232RL-REEL U?
+L dk_Interface-Controllers:FT232RL-REEL U2
 U 1 1 5DA289DB
 P 4050 2800
-F 0 "U?" H 3900 3503 60  0000 C CNN
+F 0 "U2" H 3900 3503 60  0000 C CNN
 F 1 "FT232RL-REEL" H 3900 3397 60  0000 C CNN
 F 2 "digikey-footprints:SSOP-28_W5.30mm" H 4250 3000 60  0001 L CNN
@@
 	1250 7150 1250 5750
 Wire Notes Line
-	7300 2750 7300 4600
-Wire Notes Line
-	7300 4600 10300 4600
-Wire Notes Line
-	10300 4600 10300 2750
-Wire Notes Line
-	10300 2750 7300 2750
-Text Notes 10300 2850 2    50   Italic 10
+	7400 1050 7400 2900
+Wire Notes Line
+	7400 2900 10400 2900
+Wire Notes Line
+	10400 2900 10400 1050
+Wire Notes Line
+	10400 1050 7400 1050
+Text Notes 10400 1150 2    50   Italic 10
 eZ80 Port D UART
 Text Notes 5750 1150 2    50   Italic 10
@@
 Text Notes 3250 5850 2    50   Italic 10
 Serial Traffic Indicators
-Text Notes 7900 4400 0    50   ~ 0
-Note: JTAG debug header is in the backplane\nsheet!
+Text Notes 8000 2700 0    50   ~ 0
+Note: ZDI debug header is in the backplane\nsheet!
+Wire Wire Line
+	2150 2700 2150 3000
+Wire Wire Line
+	1850 3100 1850 3000
+Wire Wire Line
+	1850 2900 1850 3000
+Connection ~ 1850 3000
+Wire Wire Line
+	1850 3000 2150 3000
 $EndSCHEMATC

Commit message: System management, serial I/O, and power refinement
  - Swapped the XTAL for the CPU to the programmable OSC.
  - Cleaned up the decoupling caps according to datasheets
    and "rule of thumb" experimental results in
    https://www.edn.com/design/components-and-packaging/4351231/EDN-Access-09-01-95-Don-t-let-rules-of-thumb-set-decoupling-capacitor-value
  - Added an ATMega328 for use as a system management uC.
    Primarily used for soft power on/off of the ATX PSU
    and control the state of /RESET during power on.
  - Reorganized the top level sheet to better illustrate
    the relationships between sheets.
  - Added an additional FT232 USB->UART IC for use with
    the SMC uC.
Parts:
- added C29, C30, C34: 100nF, symbol Device:C_Small
- added C33: 4.7uF, symbol Device:CP1_Small
- added J7: USB_B_Micro, symbol Connector:USB_B_Micro
- added J8: ZDI, symbol Connector_Generic:Conn_02x03_Odd_Even
- added R1, R10, R9: 10K, symbol Device:R_Small_US
- added R2: 4.7K, symbol Device:R_Small_US
- added U5: FT232RL-REEL, digikey-footprints:SSOP-28_W5.30mm, symbol dk_Interface-Controllers:FT232RL-REEL
Connections:
- net labels added: +3.3V, SMC_RXD, SMC_TXD, ZDI_TCK, ZDI_TDI
- wire segments 54 -> 111
- no-connect marks 14 -> 27
Other:
- note added: "USB->SMC UART Interface"
- note added: "USB->eZ80 UART Interface"
- note added: "ZDI Debug Header"
- note removed: "FT232RL USB->UART Interface"
- note removed: "Note: ZDI debug header is in the backplane\nsheet!"
- moved on the sheet: R5, R6, R7, R8

Commit message: Bookmark of where I'm at in the layout.
Last step for the serial debug interface is to route the RX/TX
lines through the opto-isolators and then to the eZ80 and the
supervisor uC.
Parts:
- removed C26, C28, C29, C30, C34: 100nF, symbol Device:C_Small
- removed C27, C33: 4.7uF, symbol Device:CP1_Small
- removed J7: USB_B_Micro, symbol Connector:USB_B_Micro
- removed R2, R8: 4.7K, symbol Device:R_Small_US
- removed R7: 10K, symbol Device:R_Small_US
- removed U2, U5: FT232RL-REEL, digikey-footprints:SSOP-28_W5.30mm, symbol dk_Interface-Controllers:FT232RL-REEL
- added C? (x3): 0.1uF, symbol Device:C_Small
- added C? (x2): 27pF, symbol Device:C_Small
- added C?: 10uF, symbol Device:CP1_Small
- added FB?: errite_Bead_Small, symbol Device:Ferrite_Bead_Small
- added R?: 1.5K, symbol Device:R_Small_US
- added R? (x2): 27 Ohm, symbol Device:R_Small_US
- added U2: FT2232D-REEL, digikey-footprints:LQFP-48_7x7mm, symbol dk_Interface-Controllers:FT2232D-REEL
- added U? (x9): HCPL-0530, symbol Zippy:HCPL-0530
- added Y?: 6MHz, symbol Device:Crystal_Small
- C25: value 100nF -> 33nF
- J4: value USB_B_Micro -> CPU DEBUG
- R1: value 10K -> 470 Ohm
Connections:
- net labels added: +3V3, ARXD, ATXD, ATXDEN, BRXD, BTXD, BTXDEN, D+, D-, USBGND, VBUS, ~ACTS, ~ADCD, ~ADSR, ~ADTR, ~ARI, ~ARTS, ~ARXLED, ~ASLEEP, ~ATXLED, ~BCTS, ~BDCD, ~BDSR, ~BDTR, ~BRI, ~BRTS, ~BSLEEP
- net labels removed: +3.3V, SER_D+, SER_D-, SER_RES, SMC_RXD, SMC_TXD
- wire segments 111 -> 118
- no-connect marks 27 -> 16
Other:
- note added: "USB UART Debug Interface"
- note removed: "USB->SMC UART Interface"
- note removed: "USB->eZ80 UART Interface"
- moved on the sheet: R10, R5, R6, R9
