File: serial-io.sch (KiCad schematic (older format))
At the start: 32 parts, among them J4 CPU DEBUG, J8 ZDI, U1 EZ80L92AZ050SG, U2 FT2232D-REEL

Commit message: debug: First draft of opto-isolation
This is the first pass of integrating opto isolators into the
debug conectors for the board.
Parts:
- added C34, C43, C44: 0.1uF, symbol Device:C_Small
- added D6: RED, symbol Device:LED
- added D7: GREEN, symbol Device:LED
- added R7, R8: 270, symbol Device:R_Small_US
- gave numbers to parts that had none: 14
Connections:
- net labels added: SMC_RXD, SMC_TXD, ~BRXLED, ~BTXLED, ~CPU_CTS, ~CPU_RTS
- net labels removed: +5V, CPU_CTS, CPU_RTS, ~RXLED, ~TXLED
- wire segments 118 -> 177
- no-connect marks 16 -> 24
Other:
- note added: "Opto-isolation to SMC (B channel)"
- note added: "Opto-isolation to eZ80 (A channel)"
- note added: "Opto-isolator Power"
- note added: "USB Serial Debug Connector"
- note added: "USB UART Power"
- moved on the sheet: R1, R10, R18, R19, R2, R5, R6, R9
