File: cpu-and-backplane.sch (KiCad schematic (older format))
At the start: 2 parts

Commit message: Import of the major redesign and most of the schematic.
Changed lines of the file:
@@
 Text Label 1900 4350 0    50   ~ 0
 RTC_XOUT
-Text Label 1900 5050 0    50   ~ 0
-~RESET
 Wire Wire Line
 	3700 3350 4050 3350
@@
 Text Label 8950 2350 0    50   ~ 0
 SCL
-Text Label 8950 2500 0    50   ~ 0
-~RESET
 Wire Wire Line
 	3700 5050 4050 5050
-Text Label 4050 5050 2    50   ~ 0
-CLK
-Text Label 8950 2650 0    50   ~ 0
-CLK
-Wire Bus Line
-	3950 2150 3950 2550
-Wire Bus Line
-	3950 950  3950 2050
-Wire Bus Line
-	2050 950  2050 3650
 Text Notes 5350 3700 2    50   Italic 10
 FIXME: HALT_SLP NEEDED FOR WAKEUP!
@@
 Text Notes 4150 3550 0    50   Italic 10
 FIXME: NO ROUTING FOR ~WAIT
+Wire Bus Line
+	3950 2150 3950 2550
+Wire Bus Line
+	3950 950  3950 2050
+Wire Bus Line
+	2050 950  2050 3650
+Text HLabel 1900 5050 0    50   Input ~ 0
+~RESET
+Text HLabel 8950 2500 0    50   Input ~ 0
+~RESET
+Text HLabel 4050 5050 2    50   Input ~ 0
+CLK
+Text HLabel 8950 2650 0    50   Input ~ 0
+CLK
 $EndSCHEMATC

Commit message: Crowbar updates and ERC fixes
This updates the Crowbar bus connectors and the layout of the
schematic to match the finalized pinouts. It also corrects an
error in the original schematic where the buses were not
properly routing due to lack of labels.

Finally, this change includes fixes for the ERC and adds the CPU
and RTC crystals to the system.
Parts:
- removed J?: JTAG_HEADER, digikey-footprints:PinHeader_1x5_P2.5mm_Drill1.1mm, symbol dk_Rectangular-Connectors-Headers-Male-Pins:B5B-XH-A_LF__SN_
- added C29, C30: 22pF, symbol Device:C_Small
- added C31, C32: 18pF, symbol Device:C_Small
- added J1: ZDI, symbol Connector_Generic:Conn_02x03_Odd_Even
- added R1, R2: 10K, symbol Device:R_Small_US
- added R10, R12: 220, symbol Device:R_Small_US
- added R11, R9: 100K, symbol Device:R_Small_US
- added Y1: 20MHz Par. Fund., symbol Device:Crystal_Small
- added Y2: 32kHz Par. Fund., symbol Device:Crystal_Small
- gave numbers to parts that had none: 1
Connections:
- net labels added: +3.3V, ADDR0, ADDR1, ADDR10, ADDR11, ADDR12, ADDR13, ADDR14, ADDR15, ADDR16, ADDR17, ADDR18, ADDR19, ADDR2, ADDR20, ADDR21, ADDR22, ADDR23, ADDR3, ADDR4, ADDR5, ADDR6, ADDR7, ADDR8, ADDR9, DATA0, DATA1, DATA2, DATA3, DATA4, DATA5, DATA6, DATA7, GND, PHI, TCK, TDI, ~CS0, ~CS1, ~CS2, ~CS3
- net labels removed: CLK, JTAG_TCK, JTAG_TDI, JTAG_TDO, JTAG_TMS, JTAG_TRIGOUT, SCL, SDA, ~IORQ
- wire segments 72 -> 118
- no-connect marks 1 -> 5
Other:
- note added: "CPU / System Clock"
- note added: "FIXME: ROUTE ON MAINBOARD ONLY"
- note added: "FIXME: ROUTE TO MAINBOARD ONLY"
- note added: "FIXME: ROUTE TO SYSTEM RAM"
- note added: "NOTE: NO MORE THAN 4pF STRAY CAPACITANCE"
- note added: "RTC Clock"
- note added: "ZDI Debug Interface"
- note removed: "FIXME: CLK from XTAL instead of PHI?"
- note removed: "FIXME: CPU CRYSTAL"
- note removed: "FIXME: HALT_SLP NEEDED FOR WAKEUP!"
- note removed: "FIXME: NO ROUTING FOR CS[0..3]"
- note removed: "FIXME: NO ROUTING FOR NMI?"
- note removed: "FIXME: NO ROUTING FOR ~INSTRD?"
- note removed: "FIXME: NO ROUTING FOR ~WAIT"
- note removed: "FIXME: RTC CRYSTAL"

Commit message: System management, serial I/O, and power refinement
  - Swapped the XTAL for the CPU to the programmable OSC.
  - Cleaned up the decoupling caps according to datasheets
    and "rule of thumb" experimental results in
    https://www.edn.com/design/components-and-packaging/4351231/EDN-Access-09-01-95-Don-t-let-rules-of-thumb-set-decoupling-capacitor-value
  - Added an ATMega328 for use as a system management uC.
    Primarily used for soft power on/off of the ATX PSU
    and control the state of /RESET during power on.
  - Reorganized the top level sheet to better illustrate
    the relationships between sheets.
  - Added an additional FT232 USB->UART IC for use with
    the SMC uC.
Parts:
- removed C29, C30: 22pF, symbol Device:C_Small
- removed J1: ZDI, symbol Connector_Generic:Conn_02x03_Odd_Even
- removed R1, R2: 10K, symbol Device:R_Small_US
- removed R10: 220, symbol Device:R_Small_US
- removed R9: 100K, symbol Device:R_Small_US
- removed Y1: 20MHz Par. Fund., symbol Device:Crystal_Small
- added X1: GR-8002DC-PCB, symbol Zippy:GR-8002DC-PTB
Connections:
- net labels added: +3V3, CROWBAR_SCL, CROWBAR_SDA, SYS_CLK, ZDI_TCK, ZDI_TDI
- net labels removed: +3.3V, CPU_XIN, CPU_XOUT, I2C_SCL, I2C_SDA, TCK, TDI
- wire segments 118 -> 91
Other:
- note added: "Programmed to 50MHz, socketed DIP half size"
- note removed: "FIXME: DO WE NEED A RESET CONTROLLER?"
- note removed: "FIXME: ROUTE ON MAINBOARD ONLY"
- note removed: "ZDI Debug Interface"
- moved on the sheet: R11, R12

Commit message: Cleanups and pruning
  - Migrated the Crowbar backplane out to the top level and
    promoted most of the signals to hierarchical labels.
  - Added a sheet for memory. Just a placeholder for now.
  - Wired up all the rest of the signals properly.
Parts:
- added unit 3 of U1
- added unit 4 of U1
Connections:
- net labels added: CPU_CLK
- net labels removed: SYS_CLK, ~IRQ0, ~IRQ1
- wire segments 91 -> 77
- no-connect marks 5 -> 21
Other:
- note added: "CPU Clock"
- note added: "eZ80L92 CPU Logic"
- note removed: "CPU / System Clock"
- moved on the sheet: R11, R12, X1

Commit message: crowbar: Reworking the pinout again
  - Completely reworked the pinout of the crowbar bus to match the
    spec.
  - Added lines for eZ80 -> SMC I2C
  - Added lines for SMC -> Crowbar I2C
  - Migrated Crowbar power pinouts to their own sub-sheet
Connections:
- net labels added: SMC_SCL, SMC_SDA, SPI_MISO, SPI_MOSI, SPI_SCLK
- net labels removed: CROWBAR_SCL, CROWBAR_SDA
- wire segments 77 -> 80
- no-connect marks 21 -> 18
Changed lines of the file:
@@
 $Descr A4 11693 8268
 encoding utf-8
-Sheet 2 7
+Sheet 2 8
 Title ""
 Date ""
@@
 ~NMI
 Text HLabel 2400 4050 0    50   Input ~ 0
-CROWBAR_SCL
+SMC_SCL
 Text HLabel 2400 4150 0    50   Input ~ 0
-CROWBAR_SDA
+SMC_SDA
 Wire Notes Line
 	1450 800  6200 800
@@
 NoConn ~ 4600 5700
 NoConn ~ 4600 5800
-NoConn ~ 4600 5900
 NoConn ~ 4600 6000
 NoConn ~ 4600 6100
-NoConn ~ 4600 6200
-NoConn ~ 4600 6300
 Text HLabel 4550 2950 2    50   Input ~ 0
 ~IOREQ
@@
 Text HLabel 4550 4050 2    50   Input ~ 0
 ~BUSACK
+Wire Wire Line
+	4600 5900 4850 5900
+Wire Wire Line
+	4600 6200 4850 6200
+Wire Wire Line
+	4600 6300 4850 6300
 Wire Bus Line
 	4700 2250 4700 2650
@@
 Wire Bus Line
 	2150 1050 2150 3750
+Text HLabel 4850 5900 2    50   Input ~ 0
+SPI_SCLK
+Text HLabel 4850 6200 2    50   Input ~ 0
+SPI_MISO
+Text HLabel 4850 6300 2    50   Input ~ 0
+SPI_MOSI
 $EndSCHEMATC

Commit message: toplevel: Add in SPI_SSx, IRQx, and INSTRD
  - Create the SPI_SSx and IRQx pins in the CPU schematic
  - Create the INSTRD pin in the memory schematic
  - Wire things up on the toplevel
Connections:
- net labels added: ~IRQ0, ~IRQ1, ~IRQ2, ~IRQ3, ~SPI_SS0, ~SPI_SS1, ~SPI_SS2, ~SPI_SS3
Changed lines of the file:
@@
 Wire Wire Line
 	4600 6300 4850 6300
+Text HLabel 4850 5900 2    50   Input ~ 0
+SPI_SCLK
+Text HLabel 4850 6200 2    50   Input ~ 0
+SPI_MISO
+Text HLabel 4850 6300 2    50   Input ~ 0
+SPI_MOSI
+Text HLabel 7350 3400 2    50   Input ~ 0
+~IRQ0
+Text HLabel 7350 3500 2    50   Input ~ 0
+~IRQ1
+Text HLabel 7350 3600 2    50   Input ~ 0
+~IRQ2
+Text HLabel 7350 3700 2    50   Input ~ 0
+~IRQ3
+Text HLabel 7350 3950 2    50   Input ~ 0
+~SPI_SS0
+Text HLabel 7350 4050 2    50   Input ~ 0
+~SPI_SS1
+Text HLabel 7350 4150 2    50   Input ~ 0
+~SPI_SS2
+Text HLabel 7350 4250 2    50   Input ~ 0
+~SPI_SS3
 Wire Bus Line
 	4700 2250 4700 2650
@@
 Wire Bus Line
 	2150 1050 2150 3750
-Text HLabel 4850 5900 2    50   Input ~ 0
-SPI_SCLK
-Text HLabel 4850 6200 2    50   Input ~ 0
-SPI_MISO
-Text HLabel 4850 6300 2    50   Input ~ 0
-SPI_MOSI
 $EndSCHEMATC

Commit message: crowbar: Wire in INTx and SPI_SSx
This wires in the INTx lines into the B port, with the SPI_SSx
lines tied into the upper bits of the B port as well.
Parts:
- added R?: 220, symbol Device:R_Small_US
Connections:
- wire segments 80 -> 91
- no-connect marks 18 -> 9
Changed lines of the file:
@@
 	-1   0    0    -1
 $EndComp
-NoConn ~ 2400 5600
-NoConn ~ 2400 5700
-NoConn ~ 2400 5800
-NoConn ~ 2400 5900
-NoConn ~ 2400 6000
-NoConn ~ 2400 6100
-NoConn ~ 2400 6200
-NoConn ~ 2400 6300
 NoConn ~ 4600 5600
 NoConn ~ 4600 5700
-NoConn ~ 4600 5800
 NoConn ~ 4600 6000
 NoConn ~ 4600 6100
@@
 ~BUSACK
 Wire Wire Line
-	4600 5900 4850 5900
+	4600 5900 4700 5900
 Wire Wire Line
-	4600 6200 4850 6200
+	4600 6200 4700 6200
 Wire Wire Line
-	4600 6300 4850 6300
-Text HLabel 4850 5900 2    50   Input ~ 0
+	4600 6300 4700 6300
+Text HLabel 4700 5900 2    50   Input ~ 0
 SPI_SCLK
-Text HLabel 4850 6200 2    50   Input ~ 0
+Text HLabel 4700 6200 2    50   Input ~ 0
 SPI_MISO
-Text HLabel 4850 6300 2    50   Input ~ 0
+Text HLabel 4700 6300 2    50   Input ~ 0
 SPI_MOSI
-Text HLabel 7350 3400 2    50   Input ~ 0
+Text HLabel 2300 5600 0    50   Input ~ 0
 ~IRQ0
-Text HLabel 7350 3500 2    50   Input ~ 0
+Text HLabel 2300 5700 0    50   Input ~ 0
 ~IRQ1
-Text HLabel 7350 3600 2    50   Input ~ 0
+Text HLabel 2300 5800 0    50   Input ~ 0
 ~IRQ2
-Text HLabel 7350 3700 2    50   Input ~ 0
+Text HLabel 2300 5900 0    50   Input ~ 0
 ~IRQ3
-Text HLabel 7350 3950 2    50   Input ~ 0
+Text HLabel 2300 6000 0    50   Input ~ 0
 ~SPI_SS0
-Text HLabel 7350 4050 2    50   Input ~ 0
+Text HLabel 2300 6100 0    50   Input ~ 0
 ~SPI_SS1
-Text HLabel 7350 4150 2    50   Input ~ 0
+Text HLabel 2300 6200 0    50   Input ~ 0
 ~SPI_SS2
-Text HLabel 7350 4250 2    50   Input ~ 0
+Text HLabel 2300 6300 0    50   Input ~ 0
 ~SPI_SS3
+Wire Wire Line
+	2400 5600 2300 5600
+Wire Wire Line
+	2400 5700 2300 5700
+Wire Wire Line
+	2400 5800 2300 5800
+Wire Wire Line
+	2400 5900 2300 5900
+Wire Wire Line
+	2400 6000 2300 6000
+Wire Wire Line
+	2400 6100 2300 6100
+Wire Wire Line
+	2400 6200 2300 6200
+Wire Wire Line
+	2400 6300 2300 6300
+Wire Wire Line
+	4600 5800 4900 5800
+Wire Wire Line
+	4900 5800 4900 5750
+$Comp
+L Device:R_Small_US R?
+U 1 1 5DAD1D17
+P 4900 5650
+F 0 "R?" H 4968 5696 50  0000 L CNN
+F 1 "220" H 4968 5605 50  0000 L CNN
+F 2 "" H 4900 5650 50  0001 C CNN
+F 3 "~" H 4900 5650 50  0001 C CNN
+	1    4900 5650
+	1    0    0    -1
+$EndComp
+$Comp
+L power:+3V3 #PWR?
+U 1 1 5DAD60C5
+P 4900 5500
+F 0 "#PWR?" H 4900 5350 50  0001 C CNN
+F 1 "+3V3" H 4915 5673 50  0000 C CNN
+F 2 "" H 4900 5500 50  0001 C CNN
+F 3 "" H 4900 5500 50  0001 C CNN
+	1    4900 5500
+	1    0    0    -1
+$EndComp
+Wire Wire Line
+	4900 5500 4900 5550
 Wire Bus Line
 	4700 2250 4700 2650
