File: backplane-connnectors.sch (KiCad schematic (older format))
At the start: 20 parts

Commit message: Crowbar updates and ERC fixes
This updates the Crowbar bus connectors and the layout of the
schematic to match the finalized pinouts. It also corrects an
error in the original schematic where the buses were not
properly routing due to lack of labels.

Finally, this change includes fixes for the ERC and adds the CPU
and RTC crystals to the system.
Parts:
- gave numbers to parts that had none: 16
Connections:
- net labels added: ADDR0, ADDR1, ADDR10, ADDR11, ADDR12, ADDR13, ADDR14, ADDR15, ADDR16, ADDR17, ADDR18, ADDR19, ADDR2, ADDR20, ADDR21, ADDR22, ADDR23, ADDR3, ADDR4, ADDR5, ADDR6, ADDR7, ADDR8, ADDR9, DATA0, DATA1, DATA2, DATA3, DATA4, DATA5, DATA6, DATA7, PHI, ~CS3, ~WAIT
- net labels removed: CLK
- wire segments 128 -> 252
Other:
- note removed: "FIXME: I2C IS ACTIVE LOW?!"
- note removed: "FIXME: RST IS ACTIVE LOW?"
- note removed: "FIXME: STOP USING 3V3 AND\nGND HERE! IF IT SHORTS IT\nWILL SLAG THE BOARD!"

Commit message: System management, serial I/O, and power refinement
  - Swapped the XTAL for the CPU to the programmable OSC.
  - Cleaned up the decoupling caps according to datasheets
    and "rule of thumb" experimental results in
    https://www.edn.com/design/components-and-packaging/4351231/EDN-Access-09-01-95-Don-t-let-rules-of-thumb-set-decoupling-capacitor-value
  - Added an ATMega328 for use as a system management uC.
    Primarily used for soft power on/off of the ATX PSU
    and control the state of /RESET during power on.
  - Reorganized the top level sheet to better illustrate
    the relationships between sheets.
  - Added an additional FT232 USB->UART IC for use with
    the SMC uC.
Parts:
- removed C1, C13, C5, C9: 10nF, symbol Device:CP1_Small
- removed C10, C11, C12, C14, C15, C16, C2, C3, C4, C6, C7, C8: 4.7uF, symbol Device:CP1_Small
- added C? (x16): 10nF, symbol Device:C_Small
Other:
- note removed: "FIXME: CALCULATE ACTUAL CAP VALUES!"
- note removed: "FIXME: DO WE *NEED* ELECTROLYTIC?"

Commit message: Cleanups and pruning
  - Migrated the Crowbar backplane out to the top level and
    promoted most of the signals to hierarchical labels.
  - Added a sheet for memory. Just a placeholder for now.
  - Wired up all the rest of the signals properly.
Parts:
- gave numbers to parts that had none: 16
Connections:
- net labels added: ~CS[0..3], ~RESET
- net labels removed: RST
- wire segments 252 -> 256

Commit message: crowbar: Reworking the pinout again
  - Completely reworked the pinout of the crowbar bus to match the
    spec.
  - Added lines for eZ80 -> SMC I2C
  - Added lines for SMC -> Crowbar I2C
  - Migrated Crowbar power pinouts to their own sub-sheet
Parts:
- removed C1, C10, C11, C12, C13, C14, C15, C16, C2, C3, C4, C5, C6, C7, C8, C9: 10nF, symbol Device:C_Small
- removed unit 2 of CR1
- removed CR2: Crowbar_Connector, symbol Zippy:Crowbar_Connector
- removed unit 2 of CR3
- removed unit 2 of CR4
- added CR3: Crowbar SLOT 2, symbol Zippy:Crowbar_Connector
- added R? (x2): 2KΩ, symbol Device:R_Small_US
- CR1: value Crowbar_Connector -> Crowbar SLOT 0
- CR3: value Crowbar_Connector -> Crowbar SLOT 1
- CR4: value Crowbar_Connector -> Crowbar SLOT 3
Connections:
- net labels added: CROWBAR_SCL, CROWBAR_SDA, SPI_MISO, SPI_MOSI, SPI_SCLK, ~IRQ2, ~IRQ3, ~SPI_SS0, ~SPI_SS1, ~SPI_SS2, ~SPI_SS3
- net labels removed: +12V, SCL, SDA
- wire segments 256 -> 234
Other:
- note added: "Crowbar Slot Connectors"
- note added: "I2C Pullups"
- note removed: "Crowbar Bus Signal and ID Pins"
- note removed: "Crowbar Power Distribution and Filtering"

Commit message: Major rework of the system RAM integration   - Wired up the jellybean logic for the RAM chip selects.   - Reorganized various bits here and there.   - Added preliminary symbols for the jellybean logic.
Connections:
- net labels added: ~IRQ[0..3], ~SLOT_CS0, ~SLOT_CS1, ~SLOT_CS2, ~SLOT_CS3, ~SLOT_CS[0..3], ~SPI_SS[0..3]
- net labels removed: ~CS3, ~CS[0..3]
- wire segments 234 -> 238
Other:
- note removed: "Crowbar Slot Connectors"
- moved on the sheet: R?
