File: power-rails.sch (KiCad schematic (older format))
At the start: 16 parts

Commit message: Crowbar updates and ERC fixes
This updates the Crowbar bus connectors and the layout of the
schematic to match the finalized pinouts. It also corrects an
error in the original schematic where the buses were not
properly routing due to lack of labels.

Finally, this change includes fixes for the ERC and adds the CPU
and RTC crystals to the system.
Parts:
- gave numbers to parts that had none: 14
- renumbered PWR_OK to PWR_OK1, PWR_ON to PWR_ON1
Connections:
- net labels added: +3.3V
- net labels removed: BATT
- wire segments 116 -> 117
Other:
- note added: "ERC Flags"
- note added: "FIXME: Is this how ATX does ~PS_ON?"
- note removed: "FIXME: Is this ATX correct?"

Commit message: System management, serial I/O, and power refinement
  - Swapped the XTAL for the CPU to the programmable OSC.
  - Cleaned up the decoupling caps according to datasheets
    and "rule of thumb" experimental results in
    https://www.edn.com/design/components-and-packaging/4351231/EDN-Access-09-01-95-Don-t-let-rules-of-thumb-set-decoupling-capacitor-value
  - Added an ATMega328 for use as a system management uC.
    Primarily used for soft power on/off of the ATX PSU
    and control the state of /RESET during power on.
  - Reorganized the top level sheet to better illustrate
    the relationships between sheets.
  - Added an additional FT232 USB->UART IC for use with
    the SMC uC.
Parts:
- removed C17, C18, C19, C20, C21, C22, C23, C24: 0.1uF, symbol Device:C_Small
- removed J2: PWR, digikey-footprints:PinHeader_1x2_P2.54mm_Drill1.02mm, symbol dk_Rectangular-Connectors-Headers-Male-Pins:22-23-2021
- added C? (x2): 1.0uF, symbol Device:C_Small
- added C? (x8): 10nF, symbol Device:C_Small
- added U3: AZ1117-3.3, symbol Regulator_Linear:AZ1117-3.3
Connections:
- net labels added: +3V3SB
- wire segments 117 -> 124
Other:
- note added: "System Management +3V3 Standby"
- note removed: "FIXME: Is this how ATX does ~PS_ON?"
- note removed: "To ATX\npower switch"
Changed lines of the file:
@@
 $Descr A4 11693 8268
 encoding utf-8
-Sheet 4 5
+Sheet 4 6
 Title ""
 Date ""
@@
 	-1   0    0    1
 $EndComp
-Text HLabel 1950 3250 0    50   Input ~ 0
-5VSB
 $Comp
 L power:+12V #PWR0127
@@
 	1    6550 1450
 	1    0    0    -1
-$EndComp
-$Comp
-L Device:C_Small C20
-U 1 1 5D90F670
-P 6750 2650
-F 0 "C20" V 6521 2650 50  0000 C CNN
-F 1 "0.1uF" V 6612 2650 50  0000 C CNN
-F 2 "" H 6750 2650 50  0001 C CNN
-F 3 "~" H 6750 2650 50  0001 C CNN
-	1    6750 2650
-	0    1    1    0
-$EndComp
-$Comp
-L Device:C_Small C21
-U 1 1 5D92D1C9
-P 6750 3000
-F 0 "C21" V 6521 3000 50  0000 C CNN
-F 1 "0.1uF" V 6612 3000 50  0000 C CNN
-F 2 "" H 6750 3000 50  0001 C CNN
-F 3 "~" H 6750 3000 50  0001 C CNN
-	1    6750 3000
-	0    1    1    0
-$EndComp
-$Comp
-L Device:C_Small C22
-U 1 1 5D92D8D1
-P 6750 3350
-F 0 "C22" V 6521 3350 50  0000 C CNN
-F 1 "0.1uF" V 6612 3350 50  0000 C CNN
-F 2 "" H 6750 3350 50  0001 C CNN
-F 3 "~" H 6750 3350 50  0001 C CNN
-	1    6750 3350
-	0    1    1    0
-$EndComp
-$Comp
-L Device:C_Small C23
-U 1 1 5D92DE52
-P 6750 3700
-F 0 "C23" V 6521 3700 50  0000 C CNN
-F 1 "0.1uF" V 6612 3700 50  0000 C CNN
-F 2 "" H 6750 3700 50  0001 C CNN
-F 3 "~" H 6750 3700 50  0001 C CNN
-	1    6750 3700
-	0    1    1    0
-$EndComp
-$Comp
-L Device:C_Small C24
-U 1 1 5D92E360
-P 6750 4050
-F 0 "C24" V 6521 4050 50  0000 C CNN
-F 1 "0.1uF" V 6612 4050 50  0000 C CNN
-F 2 "" H 6750 4050 50  0001 C CNN
-F 3 "~" H 6750 4050 50  0001 C CNN
-	1    6750 4050
-	0    1    1    0
-$EndComp
-$Comp
-L Device:C_Small C19
-U 1 1 5D934A00
-P 6750 2300
-F 0 "C19" V 6521 2300 50  0000 C CNN
-F 1 "0.1uF" V 6612 2300 50  0000 C CNN
-F 2 "" H 6750 2300 50  0001 C CNN
-F 3 "~" H 6750 2300 50  0001 C CNN
-	1    6750 2300
-	0    1    1    0
-$EndComp
-$Comp
-L Device:C_Small C18
-U 1 1 5D9352CA
-P 6750 1950
-F 0 "C18" V 6521 1950 50  0000 C CNN
-F 1 "0.1uF" V 6612 1950 50  0000 C CNN
-F 2 "" H 6750 1950 50  0001 C CNN
-F 3 "~" H 6750 1950 50  0001 C CNN
-	1    6750 1950
-	0    1    1    0
-$EndComp
-$Comp
-L Device:C_Small C17
-U 1 1 5D9356AD
-P 6750 1600
-F 0 "C17" H 6521 1600 50  0000 C CNN
-F 1 "0.1uF" V 6612 1600 50  0000 C CNN
-F 2 "" H 6750 1600 50  0001 C CNN
-F 3 "~" H 6750 1600 50  0001 C CNN
-	1    6750 1600
-	0    1    1    0
 $EndComp
 $Comp
@@
 eZ80 Power Rails
 Wire Notes Line
-	1400 5500 1400 1550
+	1400 5100 1400 1550
 Wire Notes Line
 	1400 1550 4050 1550
@@
 Wire Wire Line
 	2050 3550 2050 3600
-$Comp
-L dk_Rectangular-Connectors-Headers-Male-Pins:22-23-2021 J2
-U 1 1 5DA90496
-P 2550 5200
-F 0 "J2" V 2549 5072 50  0000 R CNN
-F 1 "PWR" V 2640 5072 50  0000 R CNN
-F 2 "digikey-footprints:PinHeader_1x2_P2.54mm_Drill1.02mm" H 2750 5400 60  0001 L CNN
-F 3 "https://media.digikey.com/pdf/Data%20Sheets/Molex%20PDFs/A-6373-N_Series_Dwg_2010-12-03.pdf" H 2750 5500 60  0001 L CNN
-F 4 "WM4200-ND" H 2750 5600 60  0001 L CNN "Digi-Key_PN"
-F 5 "22-23-2021" H 2750 5700 60  0001 L CNN "MPN"
-F 6 "Connectors, Interconnects" H 2750 5800 60  0001 L CNN "Category"
-F 7 "Rectangular Connectors - Headers, Male Pins" H 2750 5900 60  0001 L CNN "Family"
-F 8 "https://media.digikey.com/pdf/Data%20Sheets/Molex%20PDFs/A-6373-N_Series_Dwg_2010-12-03.pdf" H 2750 6000 60  0001 L CNN "DK_Datasheet_Link"
-F 9 "/product-detail/en/molex/22-23-2021/WM4200-ND/26667" H 2750 6100 60  0001 L CNN "DK_Detail_Page"
-F 10 "CONN HEADER VERT 2POS 2.54MM" H 2750 6200 60  0001 L CNN "Description"
-F 11 "Molex" H 2750 6300 60  0001 L CNN "Manufacturer"
-F 12 "Active" H 2750 6400 60  0001 L CNN "Status"
-	1    2550 5200
-	0    -1   1    0
-$EndComp
-Wire Notes Line
-	4050 1550 4050 5500
-Wire Notes Line
-	1400 5500 4050 5500
+Wire Notes Line
+	4050 1550 4050 5100
+Wire Notes Line
+	1400 5100 4050 5100
 $Comp
 L Device:LED PWR_OK1
@@
 	-1   0    0    1
 $EndComp
-Text Notes 3050 5350 0    50   ~ 0
-To ATX\npower switch
 Wire Wire Line
 	2350 4250 2050 4250
@@
 Connection ~ 3350 4650
 Wire Wire Line
-	3150 2750 3450 2750
+	3150 2750 3350 2750
 $Comp
 L power:GND #PWR0141
@@
 Wire Wire Line
 	3850 2650 3850 2700
-Text Label 3450 2750 2    50   ~ 0
-~PS_ON
-Text Label 2200 5300 0    50   ~ 0
-~PS_ON
-$Comp
-L power:GND #PWR0142
-U 1 1 5DB2739A
-P 2050 5200
-F 0 "#PWR0142" H 2050 4950 50  0001 C CNN
-F 1 "GND" V 2055 5072 50  0000 R CNN
-F 2 "" H 2050 5200 50  0001 C CNN
-F 3 "" H 2050 5200 50  0001 C CNN
-	1    2050 5200
-	0    1    1    0
-$EndComp
-Wire Wire Line
-	2450 5300 2200 5300
-Wire Wire Line
-	2050 5200 2450 5200
-Text Notes 2000 5500 0    50   Italic 10
-FIXME: Is this how ATX does ~PS_ON?
 $Comp
 L power:+3.3V #PWR0151
@@
 Wire Wire Line
 	7550 2950 7550 3050
+$Comp
+L Regulator_Linear:AZ1117-3.3 U?
+U 1 1 5D9A49ED
+P 2550 6400
+AR Path="/5D99435D/5D9A49ED" Ref="U?"  Part="1"
+AR Path="/5D86D88B/5D9A49ED" Ref="U3"  Part="1"
+F 0 "U3" H 2550 6642 50  0000 C CNN
+F 1 "AZ1117-3.3" H 2550 6551 50  0000 C CNN
+F 2 "" H 2550 6650 50  0001 C CIN
+F 3 "https://www.diodes.com/assets/Datasheets/AZ1117.pdf" H 2550 6400 50  0001 C CNN
+	1    2550 6400
+	1    0    0    -1
+$EndComp
+Text Label 1950 3250 0    50   ~ 0
+5VSB
+Text Label 1600 6400 0    50   ~ 0
+5VSB
+$Comp
+L power:GND #PWR04
+U 1 1 5D9B25B7
+P 2550 6800
+F 0 "#PWR04" H 2550 6550 50  0001 C CNN
+F 1 "GND" H 2555 6627 50  0000 C CNN
+F 2 "" H 2550 6800 50  0001 C CNN
+F 3 "" H 2550 6800 50  0001 C CNN
+	1    2550 6800
+	1    0    0    -1
+$EndComp
+Wire Wire Line
+	2550 6700 2550 6800
+Text GLabel 3250 6400 2    50   Input ~ 0
++3V3SB
+Wire Notes Line
+	1400 5900 3650 5900
+Wire Notes Line
+	3650 5900 3650 7150
+Wire Notes Line
+	3650 7150 1400 7150
+Wire Notes Line
+	1400 7150 1400 5900
+Text Notes 3650 6000 2    50   Italic 10
+System Management +3V3 Standby
+Wire Wire Line
+	2850 6400 3000 6400
+Text HLabel 3350 2750 2    50   Input ~ 0
+~PS_ON
+$Comp
+L power:PWR_FLAG #FLG0104
+U 1 1 5DC7B5E2
+P 1600 6400
+F 0 "#FLG0104" H 1600 6475 50  0001 C CNN
+F 1 "PWR_FLAG" H 1600 6573 50  0000 C CNN
+F 2 "" H 1600 6400 50  0001 C CNN
+F 3 "~" H 1600 6400 50  0001 C CNN
+	1    1600 6400
+	-1   0    0    1
+$EndComp
+Wire Wire Line
+	1600 6400 2000 6400
+$Comp
+L Device:C_Small C?
+U 1 1 5DCF8440
+P 2000 6600
+F 0 "C?" H 2092 6646 50  0000 L CNN
+F 1 "1.0uF" H 2092 6555 50  0000 L CNN
+F 2 "" H 2000 6600 50  0001 C CNN
+F 3 "~" H 2000 6600 50  0001 C CNN
+	1    2000 6600
+	1    0    0    -1
+$EndComp
+$Comp
+L Device:C_Small C?
+U 1 1 5DCF8E1D
+P 3000 6600
+F 0 "C?" H 3092 6646 50  0000 L CNN
+F 1 "1.0uF" H 3092 6555 50  0000 L CNN
+F 2 "" H 3000 6600 50  0001 C CNN
+F 3 "~" H 3000 6600 50  0001 C CNN
+	1    3000 6600
+	1    0    0    -1
+$EndComp
+Wire Wire Line
+	2000 6500 2000 6400
+Connection ~ 2000 6400
+Wire Wire Line
+	2000 6400 2250 6400
+Wire Wire Line
+	3000 6500 3000 6400
+Connection ~ 3000 6400
+Wire Wire Line
+	3000 6400 3250 6400
+$Comp
+L power:GND #PWR?
+U 1 1 5DD012B9
+P 2000 6800
+F 0 "#PWR?" H 2000 6550 50  0001 C CNN
+F 1 "GND" H 2005 6627 50  0000 C CNN
+F 2 "" H 2000 6800 50  0001 C CNN
+F 3 "" H 2000 6800 50  0001 C CNN
+	1    2000 6800
+	1    0    0    -1
+$EndComp
+$Comp
+L power:GND #PWR?
+U 1 1 5DD017FB
+P 3000 6800
+F 0 "#PWR?" H 3000 6550 50  0001 C CNN
+F 1 "GND" H 3005 6627 50  0000 C CNN
+F 2 "" H 3000 6800 50  0001 C CNN
+F 3 "" H 3000 6800 50  0001 C CNN
+	1    3000 6800
+	1    0    0    -1
+$EndComp
+Wire Wire Line
+	2000 6800 2000 6700
+Wire Wire Line
+	3000 6800 3000 6700
+$Comp
+L Device:C_Small C?
+U 1 1 5DEEE6FB
+P 6750 1600
+F 0 "C?" V 6521 1600 50  0000 C CNN
+F 1 "10nF" V 6612 1600 50  0000 C CNN
+F 2 "" H 6750 1600 50  0001 C CNN
+F 3 "~" H 6750 1600 50  0001 C CNN
+	1    6750 1600
+	0    1    1    0
+$EndComp
+$Comp
+L Device:C_Small C?
+U 1 1 5DEEEA26
+P 6750 1950
+F 0 "C?" V 6521 1950 50  0000 C CNN
+F 1 "10nF" V 6612 1950 50  0000 C CNN
+F 2 "" H 6750 1950 50  0001 C CNN
+F 3 "~" H 6750 1950 50  0001 C CNN
+	1    6750 1950
+	0    1    1    0
+$EndComp
+$Comp
+L Device:C_Small C?
+U 1 1 5DEF3F7C
+P 6750 2300
+F 0 "C?" V 6521 2300 50  0000 C CNN
+F 1 "10nF" V 6612 2300 50  0000 C CNN
+F 2 "" H 6750 2300 50  0001 C CNN
+F 3 "~" H 6750 2300 50  0001 C CNN
+	1    6750 2300
+	0    1    1    0
+$EndComp
+$Comp
+L Device:C_Small C?
+U 1 1 5DEF3F86
+P 6750 2650
+F 0 "C?" V 6521 2650 50  0000 C CNN
+F 1 "10nF" V 6612 2650 50  0000 C CNN
+F 2 "" H 6750 2650 50  0001 C CNN
+F 3 "~" H 6750 2650 50  0001 C CNN
+	1    6750 2650
+	0    1    1    0
+$EndComp
+$Comp
+L Device:C_Small C?
+U 1 1 5DEF8BFA
+P 6750 3000
+F 0 "C?" V 6521 3000 50  0000 C CNN
+F 1 "10nF" V 6612 3000 50  0000 C CNN
+F 2 "" H 6750 3000 50  0001 C CNN
+F 3 "~" H 6750 3000 50  0001 C CNN
+	1    6750 3000
+	0    1    1    0
+$EndComp
+$Comp
+L Device:C_Small C?
+U 1 1 5DEF8C04
+P 6750 3350
+F 0 "C?" V 6521 3350 50  0000 C CNN
+F 1 "10nF" V 6612 3350 50  0000 C CNN
+F 2 "" H 6750 3350 50  0001 C CNN
+F 3 "~" H 6750 3350 50  0001 C CNN
+	1    6750 3350
+	0    1    1    0
+$EndComp
+$Comp
+L Device:C_Small C?
+U 1 1 5DEF8C0E
+P 6750 3700
+F 0 "C?" V 6521 3700 50  0000 C CNN
+F 1 "10nF" V 6612 3700 50  0000 C CNN
+F 2 "" H 6750 3700 50  0001 C CNN
+F 3 "~" H 6750 3700 50  0001 C CNN
+	1    6750 3700
+	0    1    1    0
+$EndComp
+$Comp
+L Device:C_Small C?
+U 1 1 5DEF8C18
+P 6750 4050
+F 0 "C?" V 6521 4050 50  0000 C CNN
+F 1 "10nF" V 6612 4050 50  0000 C CNN
+F 2 "" H 6750 4050 50  0001 C CNN
+F 3 "~" H 6750 4050 50  0001 C CNN
+	1    6750 4050
+	0    1    1    0
+$EndComp
 $EndSCHEMATC

Commit message: Cleanups and pruning
  - Migrated the Crowbar backplane out to the top level and
    promoted most of the signals to hierarchical labels.
  - Added a sheet for memory. Just a placeholder for now.
  - Wired up all the rest of the signals properly.
Parts:
- gave numbers to parts that had none: 10
Other:
- moved on the sheet: R3, R4

Commit message: Addition of the main bus pins to the memory sheet.
Other:
- note added: "ERC Flags and Main Power Rails"
- note removed: "ERC Flags"
Changed lines of the file:
@@
 $EndComp
 Wire Notes Line
-	6800 6600 5350 6600
-Wire Notes Line
-	5350 6600 5350 7650
-Wire Notes Line
-	5350 7650 6800 7650
+	6800 6600 4850 6600
+Wire Notes Line
+	4850 6600 4850 7650
+Wire Notes Line
+	4850 7650 6800 7650
 Wire Notes Line
 	6800 7650 6800 6600
 Text Notes 6800 6700 2    50   Italic 10
-ERC Flags
+ERC Flags and Main Power Rails
 Wire Wire Line
 	5750 3350 5750 3450
@@
 	0    1    1    0
 $EndComp
+Text GLabel 5150 7250 1    50   Input ~ 0
++3V3SB
 $EndSCHEMATC

Commit message: Bookmark of where I'm at in the layout.
Last step for the serial debug interface is to route the RX/TX
lines through the opto-isolators and then to the eZ80 and the
supervisor uC.
Parts:
- removed J3: 1-1775099-3, TE_1-1775099-3, symbol ATX_Connector:1-1775099-3
- added C41, C42: 10nF, symbol Device:CP1_Small
- added D3, D4: ???, symbol Device:D_Small
- added D5: D_Schottky_Small, symbol Device:D_Schottky_Small
- added F1: 0.5A fast, symbol Device:Fuse
- added F2: 4A fast, symbol Device:Fuse
- added J3: ATX_Connector, TE_1-1775099-3, symbol Zippy:ATX_Connector
- added L1: 18uH, symbol Device:L_Small
- added PWR_FAULT1: YELLOW, symbol Device:LED
- added R14, R15, R16, R17: 330, symbol Device:R_Small_US
- added U6: TPS3511DR, D8, symbol TPS3511DR:TPS3511DR
- added U7: AP1501A-33K5G-13, DPAK171P1524X485-6N, symbol AP1501A-33K5G-13:AP1501A-33K5G-13
- renumbered PWR_ON1 to PS_ON1
Connections:
- net labels added: ATX_12V, ATX_3V3, ATX_5V, ATX_5VSB, ATX_PWGD, PWR_GD, ~PWR_FAULT
- net labels removed: +3.3V, +5V, 5VSB, PWR_OK
- wire segments 124 -> 202
Other:
- note added: "0.5V\nDrop"
- note added: "Main +3V3 Power Rail Regulator"
- note added: "PSU Monitoring"
- note added: "System Management +3V3 Standby Rail LDO"
- note removed: "ERC Flags and Main Power Rails"
- note removed: "FIXME: Symbol pinout is horizontal rather than vertical!"
- note removed: "System Management +3V3 Standby"
- moved on the sheet: R3, R4
