File: system-management.sch (KiCad schematic (older format))
At the start: 10 parts, among them J1 RESET_BTN, J2 PWR_BTN, J5 Conn_01x03, J6 SMC_ISP, U4 ATMEGA328PB-AU

Commit message: Cleanups and pruning
  - Migrated the Crowbar backplane out to the top level and
    promoted most of the signals to hierarchical labels.
  - Added a sheet for memory. Just a placeholder for now.
  - Wired up all the rest of the signals properly.
Parts:
- gave numbers to parts that had none: 5
Other:
- note added: "ATX Front Panel Buttons"
- note added: "ISP Programming Header"
- moved on the sheet: R13

Commit message: Bookmark of where I'm at in the layout.
Last step for the serial debug interface is to route the RX/TX
lines through the opto-isolators and then to the eZ80 and the
supervisor uC.
Connections:
- net labels added: PWR_GD, ~PS_ON, ~PWR_FAULT
- net labels removed: PS_ON, PWR_OK
- wire segments 58 -> 59
- no-connect marks 11 -> 10
Changed lines of the file:
@@
 $Descr A4 11693 8268
 encoding utf-8
-Sheet 5 7
+Sheet 6 7
 Title ""
 Date ""
@@
 	3350 2950 3100 2950
 Text HLabel 3100 2950 0    50   Input ~ 0
-PS_ON
+~PS_ON
 Wire Wire Line
 	9350 4250 8850 4250
@@
 Text GLabel 4800 2550 0    50   Input ~ 0
 +3V3SB
-NoConn ~ 3350 3550
-Wire Wire Line
-	3350 3650 3100 3650
-Text HLabel 3100 3650 0    50   Input ~ 0
-PWR_OK
 NoConn ~ 3350 3750
 Text Label 1800 2300 3    50   ~ 0
@@
 Text Notes 9700 4000 2    50   Italic 10
 ATX Front Panel Buttons
+Wire Wire Line
+	3100 3550 3350 3550
+Text HLabel 3100 3550 0    50   Input ~ 0
+~PWR_FAULT
+Text HLabel 3100 3650 0    50   Input ~ 0
+PWR_GD
+Wire Wire Line
+	3350 3650 3100 3650
 $EndSCHEMATC

Commit message: debug: First draft of opto-isolation
This is the first pass of integrating opto isolators into the
debug conectors for the board.
Parts:
- J5: Notes (none) -> NORM: 1+2, PROG: 2+3
Other:
- note added: "Jumper to control programming power.\nShort pins 1+2 for normal operation.\nLAYOUT: NOTE NORMAL PINS"
- note removed: "Jumper to control programming power.\nShort pins 1+2 for normal operation."
Changed lines of the file:
@@
 EESchema Schematic File Version 4
 LIBS:Zippy-cache
-EELAYER 29 0
+EELAYER 30 0
 EELAYER END
 $Descr A4 11693 8268
@@
 F 2 "" H 5100 2700 50  0001 C CNN
 F 3 "~" H 5100 2700 50  0001 C CNN
+F 4 "NORM: 1+2, PROG: 2+3" H 5100 2700 50  0001 C CNN "Notes"
 	1    5100 2700
 	1    0    0    -1
@@
 Text Label 4400 2800 0    50   ~ 0
 PROG_PWR
-Text Notes 4350 3050 0    50   Italic 0
-Jumper to control programming power.\nShort pins 1+2 for normal operation.
+Text Notes 4350 3100 0    50   Italic 0
+Jumper to control programming power.\nShort pins 1+2 for normal operation.\nLAYOUT: NOTE NORMAL PINS
 NoConn ~ 3350 3050
 NoConn ~ 3350 3150

Commit message: Major rework of the system RAM integration   - Wired up the jellybean logic for the RAM chip selects.   - Reorganized various bits here and there.   - Added preliminary symbols for the jellybean logic.
Connections:
- net labels added: SWAP23
- wire segments 59 -> 60
- no-connect marks 10 -> 9
Changed lines of the file:
@@
 $Descr A4 11693 8268
 encoding utf-8
-Sheet 7 8
+Sheet 8 9
 Title ""
 Date ""
@@
 NoConn ~ 4150 3750
 NoConn ~ 4150 3850
-NoConn ~ 4150 3950
 NoConn ~ 4150 3250
 NoConn ~ 4150 3350
@@
 Wire Wire Line
 	3350 3650 3100 3650
+Wire Wire Line
+	4150 3950 4400 3950
+Text HLabel 4400 3950 2    50   Input ~ 0
+SWAP23
 $EndSCHEMATC
